File: simple_pa_ctl/rev-/simple_pa_ctl.brd (EAGLE design)
At the start: 88.9 x 88.9 mm, 93 parts, among them IC1 LD117ADT50TR, IC2 MCP9700, IC3 ATMEGA32U4-AU, J1 USB_B_PTH, K3 G5V1, SW1 SPST_TACT-KMR2, Y1 8MHz

Commit message: very simple, featherwing footprint
Parts:
- removed 12V, 3V3, 5V, A3, A4, A5, D7, RXLED, TP1, TXLED: TPSQTP20SQ, testpad:TP20SQ
- removed ADC1: ADS1115, vtgs:MSOP10
- removed ATTN: (no value), pinhead:1X07
- removed BTN, CASE_TEMP, FWD_REV_PWR, LCD, PA_TEMP: (no value), pinhead:1X03
- removed C1, C13, C14, C15, C16, C3: 0.1uF, rcl:C0805K
- removed C10, C12, C2, C29, C6, C7, C8, C9: 1uF, rcl:C0805K
- removed C11, C27, C28, C4, C5: 10uF, rcl:C0805K
- removed C26: 100uF, rcl:PANASONIC_D
- removed D1: MBR120, adafruit:SOD-123
- removed F1: 500mA, adafruit:R1206
- removed FAN, RELAY, THERMO: (no value), pinhead:1X02
- removed H1, H2: MOUNT-PAD-ROUND4.5, holes:4,5-PAD
- removed IC1: LD117ADT50TR, v-reg:DPACK
- removed IC2: MCP9700, vtgs:SC70
- removed IC3: ATMEGA32U4-AU, adafruit:TQFP44
- removed ICSP: (no value), pinhead:2X03
- removed J1: USB_B_PTH, SparkFun-Connectors:USB-B-PTH
- removed K3: G5V1, relay:G5V1
- removed LED5: (no value), adafruit:CHIPLED_0805
- removed R12: 220, rcl:R0805
- removed R13, R27, R28, R5, R6: 10k, rcl:R0805
- removed R30, R31, R32, R33: 1k, rcl:R0805
- removed R36, R39: 10, rcl:R0805
- removed SJ1, SJ10, SJ11, SJ12, SJ13, SJ2, SJ3, SJ4, SJ5, SJ6, SJ7, SJ9: (no value), jumper:SJ
- removed SJ14, SJ8: (no value), jumper:SJ_2
- removed SW1: SPST_TACT-KMR2, adafruit:KMR2
- removed U$2: INA260, vtgs:TSSOP16
- removed VR3: SPX3819M5_3V3, kj4qlp:SOT23-5
- removed X1: (no value), SparkFun-Retired:M25VB
- removed Y1: 8MHz, SparkFun-Clocks:RESONATOR-SMD-3.2X1.3
- added JP1: (no value), pinhead:2X04
- added MS1: FEATHERWING, adafruit:FEATHERWING
- added OC1, OC2: FOD852, vtgs:SMD4-7
- added R7, R9: 1k, rcl:R0805
- added R8: 220, rcl:R0805
- added THERMO1: (no value), pinhead:1X02
- R2: value 100k -> 220
- R3: value 22 -> 1k
- R4: value 22 -> 220
- moved R1 171.1 mm to (13.3, 17.1)
- moved LED4 156.4 mm to (42.5, 7.62), turned to 270 degrees
- moved LED3 151.1 mm to (42.5, 10.2), turned to 270 degrees
- moved LED2 146.0 mm to (42.5, 12.7), turned to 270 degrees
- moved LED1 140.9 mm to (42.5, 15.2), turned to 270 degrees
- moved OC4 137.0 mm to (28.6, 10.2), turned to 270 degrees
- moved R29 133.7 mm to (38.7, 15.2), turned to 180 degrees
- moved R3 132.8 mm to (38.7, 12.7), turned to 180 degrees
- moved OC3 125.6 mm to (23.5, 10.2), turned to 270 degrees
- moved R4 124.1 mm to (23.5, 17.1)
- moved R2 116.1 mm to (18.4, 17.1)
Connections:
- removed net +12V: 12V.TP, C26.+, C27.1, FAN.1, H2.B4,5, IC1.3, K3.2, RELAY.1, SJ14.3, U$2.14, U$2.15, U$2.16, X1.24
- removed net +3V3: 3V3.TP, ADC1.8, ATTN.6, C10.1, C11.1, C12.1, C16.1, C2.1, C5.1, C6.1, C7.1, C8.1, C9.1, CASE_TEMP.2, IC2.4, IC3.14, IC3.24, IC3.33, IC3.34, IC3.42, IC3.44, IC3.6, ICSP.2, LCD.1, LED5.A, PA_TEMP.2, R13.2, R27.2, R28.2, R5.2, R6.2, SJ11.1, SJ3.2, SJ6.2, U$2.10, VR3.5, X1.15, X1.5
- removed net +5V: 5V.TP, C4.1, D1.C, LED4.A, R2.1, SJ8.2, VR3.1, X1.7
- removed net 0_RX_THERMO: IC3.20, R13.1, THERMO.1, X1.10
- removed net 10_BUTTON_RED: BTN.1, IC3.30, R27.1, X1.21
- removed net 11_CS: IC3.12
- removed net 12_UHF_PTT_REL: IC3.26
- removed net 13_PA_PWR_REL: IC3.32, R1.1
- removed net 14_MISO_MCU: IC3.11, ICSP.1
- removed net 15_SCK: IC3.9, ICSP.3
- removed net 16_MOSI: IC3.10, ICSP.4
- removed net 1_TX: IC3.21, LCD.3, X1.8
- removed net 4_VHF_PTT_REL: IC3.25
- removed net 5_BUTTON_BLACK: BTN.2, IC3.31, R28.1, X1.9
- removed net 6_ALERT_ADC: ADC1.2, IC3.27
- removed net 8_ALERT_I: IC3.28, X1.18
- removed net 9_ALERT_T: IC3.29, X1.19
- removed net A0: SJ10.2, SJ11.2, SJ12.2, SJ13.2, U$2.5
- removed net A0_VHF_COAX_REL: IC3.36
- removed net A1: SJ5.1, SJ6.1, SJ7.1, SJ9.1, U$2.4
- removed net A1_UHF_COAX_REL: IC3.37
- removed net A2_PA_FAN: IC3.38, R12.1
- removed net A3: A3.TP, IC3.39
- removed net A4: A4.TP, IC3.40
- removed net A5: A5.TP, IC3.41
- removed net ADDR: ADC1.1, SJ1.1, SJ2.1, SJ3.1, SJ4.1
- removed net ALERT_I: U$2.7
- removed net ATTN_B0: ATTN.1
- removed net ATTN_B1: ATTN.2
- removed net ATTN_B2: ATTN.3
- removed net ATTN_B3: ATTN.4
- removed net ATTN_B4: ATTN.5
- removed net D7: D7.TP, IC3.1, LED1.A
- removed net FAN: FAN.2, K3.5, K3.6, X1.11
- removed net IN+: H1.B4,5, SJ14.1, U$2.1, U$2.2, U$2.3
- removed net N$10: IC3.4, R4.2
- removed net N$11: J1.D+, R4.1
- removed net N$16: LED1.C, R29.2
- removed net N$17: LED2.C, R30.2
- removed net N$18: LED4.C, R32.2
- removed net N$19: LED5.C, R33.2
- removed net N$21: OC4.1, R12.2
- removed net N$24: LED3.C, R31.2
- removed net N$27: OC4.3, R36.1
- removed net N$31: C28.1, C29.1, IC1.4, SJ8.3
- removed net N$39: D1.A, F1.2, SJ8.1
- removed net N$40: OC3.3, R39.1
- removed net N$9: IC3.3, R3.2
- removed net PA_PWR_REL: OC3.4, RELAY.2, X1.25
- removed net RST: IC3.13, ICSP.5, SW1.2, SW1.4
- removed net RXLED: IC3.8, LED3.A, RXLED.TP
- removed net SCL: ADC1.10, IC3.18, R5.1, SJ1.2, SJ13.1, SJ9.2, U$2.9, X1.16
- removed net SDA: ADC1.9, IC3.19, R6.1, SJ12.1, SJ2.2, SJ7.2, U$2.8, X1.17
- removed net TXLED: IC3.22, LED2.A, TXLED.TP
- removed net UHF_COAX_REL: X1.12
- removed net VBUS: C1.1, SJ14.2, U$2.12
- removed net VHF_COAX_REL: X1.13
- removed net VT_BRD: ADC1.7, C15.1, CASE_TEMP.3, IC2.3
- removed net VT_PA: ADC1.6, C14.1, PA_TEMP.3
- removed net VUSB: F1.1, IC3.7, J1.VBUS
- removed net V_FWD: ADC1.4, C13.1, FWD_REV_PWR.3, X1.2
- removed net V_REV: ADC1.5, C3.1, FWD_REV_PWR.2, X1.3
- removed net V_TEMP: X1.4
- new net !EVENT_1: JP1.1, OC1.4
- new net !EVENT_2: JP1.3, OC2.4
- new net !EVENT_3: JP1.5, OC3.4
- new net !EVENT_4: JP1.7, OC4.4
- new net GPIO_E1: MS1.25, R1.1, R29.2
- new net GPIO_E2: MS1.24, R2.1, R3.2
- new net GPIO_E3: MS1.23, R4.1, R7.2
- new net GPIO_E4: MS1.22, R8.1, R9.2
- new net N$7: OC4.1, R8.2
- net GND: now also JP1.2, JP1.4, JP1.6, JP1.8, LED1.C, LED2.C, LED3.C, LED4.C, MS1.4, OC1.2, OC1.3, OC2.2, OC2.3, OC3.3, OC4.3; no longer ADC1.3, ATTN.7, BTN.3, C1.2, C10.2, C11.2, C12.2, C13.2, C14.2, C15.2, C16.2, C2.2, C26.-, C27.2, C28.2, C29.2, C3.2, C4.2, C5.2, C6.2, C7.2, C8.2, C9.2, CASE_TEMP.1, FWD_REV_PWR.1, IC1.1, IC2.2, IC3.15, IC3.23, IC3.35, IC3.43, IC3.5, ICSP.6, J1.GND, J1.SHLD1, J1.SHLD2, K3.10, LCD.2, PA_TEMP.1, R29.1, R30.1, R31.1, R32.1, R33.1, R36.2, R39.2, SJ10.1, SJ4.2, SJ5.2, SW1.1, SW1.3, THERMO.2, TP1.TP, U$2.11, U$2.6, VR3.2, X1.1, X1.14, X1.20, X1.22, X1.23, X1.6, Y1.2
- net N$1: now also OC1.1; no longer OC3.1
- net N$2: now also LED1.A, R29.1; no longer K3.9, OC4.4
- net N$3: now also OC2.1; no longer VR3.3
- net N$4: now also LED2.A, R3.1; no longer IC3.17, Y1.1
- net N$5: now also OC3.1, R4.2; no longer IC3.16, Y1.3
- net N$6: now also LED3.A, R7.1; no longer IC2.1, IC2.5
- net N$8: now also LED4.A, R9.1; no longer J1.D-, R3.1
Routing:
- net GPIO_E1: track 0.00 -> 46.9 mm, vias 0 -> 2
- net !EVENT_1: track 0.00 -> 36.3 mm, vias 0 -> 1
- net !EVENT_2: track 0.00 -> 30.2 mm, vias 0 -> 1
- net GPIO_E2: track 0.00 -> 26.2 mm, vias 0 -> 1
- net !EVENT_3: track 0.00 -> 24.1 mm, vias 0 -> 1
- net GPIO_E3: track 0.00 -> 23.7 mm, vias 0 -> 1
- net !EVENT_4: track 0.00 -> 17.9 mm, vias 0 -> 1
- net GPIO_E4: track 0.00 -> 15.2 mm, vias 0 -> 1
- net N$1: track 0.00 -> 2.52 mm
- net N$7: track 0.00 -> 2.52 mm
- net N$5: track 0.00 -> 2.52 mm
- net N$3: track 0.00 -> 2.52 mm
- net GND: track 0.00 -> 1.24 mm, vias 0 -> 9
Other:
- board size 88.9 x 88.9 mm -> 50.8 x 22.9 mm
